File: hw/truck_stereo.kicad_pcb (KiCad board)
At the start: 2 copper layers, 43.2 x 55.9 mm, 13 parts, among them J1 Conn_01x08_Male, J2 Conn_01x08_Male, J3 Conn_01x04_Male, M1 BLUETOOTH-RN-52, U1 TPS22929D

Commit message: WIP: hw: fixups
Connections:
- B1 pad 11: Net-(B1-Pad11) -> /ROT_SW
- B1 pad 14: /ROT_SW -> Net-(B1-Pad14)
- B1 pad 22: Net-(B1-Pad22) -> /ESP32_TX
- B1 pad 23: /ESP32_TX -> Net-(B1-Pad23)
- B1 pad 24: /ESP32_RX -> Net-(B1-Pad24)
- B1 pad 25: Net-(B1-Pad25) -> /ESP32_RX
- B1 pad 29: /DISP_DC -> /DISP_CS
- B1 pad 31: /DISP_CS -> Net-(B1-Pad31)
- B1 pad 33: Net-(B1-Pad33) -> /DISP_DC
- J1 pad 6: /DISP_DC -> /DISP_CS
- J1 pad 8: /DISP_CS -> /DISP_DC
Routing:
- net /~RN52_CMD: track 29.4 -> 38.9 mm, vias 1 -> 0
- net /ROT_SW: track 7.89 -> 14.3 mm
- net /ESP32_TX: track 8.13 -> 14.2 mm
- net /ESP32_RX: track 8.13 -> 5.59 mm
- net /RN52_VDD_SW: track 34.5 -> 32.2 mm
- net /RN52_PWREN: track 46.8 -> 45.1 mm
Other:
- board text added: "Truck Stereo v1.1 Copyright 2020 Josh Watts CC BY 4.0"
- board text removed: "Truck Stereo v1.0 Copyright 2020 Josh Watts CC BY 4.0"
