File: hw/truck_stereo.sch (KiCad schematic (older format))
At the start: 16 parts, among them J1 Conn_01x08_Male, J2 Conn_01x08_Male, J3 Conn_01x04_Male, M1 BLUETOOTH-RN-52, SW1 DNP, U1 TPS22929D, U2 alpine_amp DNP

Commit message: WIP: hw: fixups
Connections:
- net DISP_CS: now also B1.29 (5), J1.6 (Pin_6); no longer B1.31 (2), J1.8 (Pin_8)
- net DISP_DC: now also B1.33 (4), J1.8 (Pin_8); no longer B1.29 (5), J1.6 (Pin_6)
- net ESP32_RX: now also B1.25 (22); no longer B1.24 (RX)
- net ESP32_TX: now also B1.22 (21); no longer B1.23 (TX)
- net ROT_SW: now also B1.11 (26); no longer B1.14 (34)
Changed lines of the file:
@@
 Text Label 9800 900  2    50   ~ 0
 REMOTE_EN
-Text Label 3050 3350 0    50   ~ 0
+Text Label 3050 3250 0    50   ~ 0
 ESP32_TX
-Text Label 3050 3450 0    50   ~ 0
+Text Label 3050 3550 0    50   ~ 0
 ESP32_RX
 Text Label 5200 4900 2    50   ~ 0
@@
 Wire Wire Line
 	1450 4650 1450 4550
-NoConn ~ 3050 3250
+NoConn ~ 3050 3350
 $Comp
 L Device:CP1_Small C1
@@
 Text Label 2050 3650 2    50   ~ 0
 ROT_B
-Text Label 2050 3750 2    50   ~ 0
+Text Label 2050 4050 2    50   ~ 0
 ROT_SW
 NoConn ~ 5200 4800
@@
 Text Label 3050 3650 0    50   ~ 0
 DISP_MISO
-Text Label 3050 4150 0    50   ~ 0
+Text Label 3050 4350 0    50   ~ 0
+DISP_DC
+Text Label 3050 3950 0    50   ~ 0
 DISP_CS
-Text Label 3050 3950 0    50   ~ 0
-DISP_DC
 Text Label 3050 4050 0    50   ~ 0
 DISP_RST
-NoConn ~ 3050 3550
+NoConn ~ 3050 3450
 Wire Wire Line
 	3050 3150 3600 3150
@@
 DISP_MISO
 Text Label 1350 850  2    50   ~ 0
+DISP_DC
+Text Label 1350 1050 2    50   ~ 0
 DISP_CS
-Text Label 1350 1050 2    50   ~ 0
-DISP_DC
 Text Label 1350 950  2    50   ~ 0
 DISP_RST
 NoConn ~ 2050 3850
-NoConn ~ 2050 4050
 Text Label 2050 4450 2    50   ~ 0
 REMOTE_EN
@@
 Text Label 2050 4550 2    50   ~ 0
 ESP32_RST
-NoConn ~ 3050 4350
+NoConn ~ 3050 4150
+NoConn ~ 2050 3750
 $EndSCHEMATC
